Commit message: tespit için worlde araba table gibi şeyler eklendi

File: yolo_bot/install/kasva_sekli/share/kasva_sekli/description/camera.xacro (robot description, xacro)
@@ -4,5 +4,5 @@
         <parent link="chassis"/>
         <child link="camera_link"/>
-        <origin xyz="0.30 0 0.2" rpy="0 0.3 0"/>  <!-- 0.35 0 0.2    0 0.18 0 -->
+        <origin xyz="0.30 0 0.2" rpy="0 0 0"/>  <!-- 0.35 0 0.2    0 0.18 0 -->
     </joint>
     <link name="camera_link">

Commit message: alma mapping de worlde düzenlemeler yaptım

File: yolo_bot/install/kasva_sekli/share/kasva_sekli/description/camera.xacro (robot description, xacro)
@@ -4,5 +4,5 @@
         <parent link="chassis"/>
         <child link="camera_link"/>
-        <origin xyz="0.30 0 0.2" rpy="0 0 0"/>  <!-- 0.35 0 0.2    0 0.18 0 -->
+        <origin xyz="0.30 0 0.2" rpy="0 0.20 0"/>  <!-- 0.35 0 0.2    0 0.18 0 -->
     </joint>
     <link name="camera_link">
